Commit message: asd

File: arm2.urdf (robot description, URDF)
Before this commit: robot oneArm, 4 links, 3 joints
Links:
- added link link0; visual cylinder length=0.01 radius=0.025
Joints:
- added joint joint0: type revolute, parent base_link, child link0, origin xyz=0 0 0.05, axis 0 0 1
- joint joint1: axis 0 0 1 -> 0 1 0; origin xyz=0 0 0.05 -> xyz=0 0 0.01; parent base_link -> link0
- joint joint2: axis 0 0 1 -> 0 1 0
- joint joint3: axis 0 0 1 -> 0 1 0
