Commit message: test

File: arm.urdf (robot description, URDF)
Before this commit: robot oneArm, 1 links, 1 joints
Links:
- added link link1

Commit message: Edited urdf

File: arm.urdf (robot description, URDF)
Before this commit: robot oneArm, 1 links, 1 joints
Links:
- added link link1
Joints:
- joint joint1: limit (none) -> effort=100 velocity=1.0

Commit message: Edited arm.urdf

File: arm.urdf (robot description, URDF)
Before this commit: robot oneArm, 2 links, 1 joints
Links:
- added link link2; visual cylinder length=0.1 radius=0.01
- added link link3; visual cylinder length=0.1 radius=0.01
- link link1: geometry visual cylinder length=0.1 radius=0.01
Joints:
- added joint joint2: type revolute, parent link1, child link2, origin xyz=0 0 0.1, axis 0 0 1
- added joint joint3: type revolute, parent link2, child link3, origin xyz=0 0 0.1, axis 0 0 1

Commit message: finished arm.urdf

File: arm.urdf (robot description, URDF)
Before this commit: robot oneArm, 4 links, 3 joints
Links:
- added link link4; visual cylinder length=0.031 radius=0.03
- added link link5; visual cylinder length=0.008 radius=0.025
- link base_link: geometry visual cylinder length=0.049 radius=0.1
- link link1: geometry visual cylinder length=0.02 radius=0.033
- link link2: geometry visual cylinder length=0.12 radius=0.03
- link link3: geometry visual cylinder length=0.127 radius=0.03
Joints:
- added joint joint4: type revolute, parent link3, child link4, origin xyz=0 0 0.127, axis 0 -1 0
- added joint joint5: type revolute, parent link4, child link5, origin xyz=0 0 0.031, axis 0 0 1
- joint joint1: origin xyz=0 0 0.1 -> xyz=0 0 0.049
- joint joint2: axis 0 0 1 -> 0 -1 0; origin xyz=0 0 0.1 -> xyz=0 0 0.02
- joint joint3: axis 0 0 1 -> 0 -1 0; origin xyz=0 0 0.1 -> xyz=0 0 0.12
